File: sw2.sch (EAGLE design)
At the start: 11 parts, among them X3 22-23-2041

Commit message: Add files via upload
Parts:
- added S1: MOMENTARY-SWITCH-SPST-PTH-6.0MM-KIT, SparkFun-Switches:MOMENTARY-SWITCH-SPST-PTH-6.0MM-KIT
Connections:
- new net N$18: ARDUINO1.RST, S1.1
- net N$4: now also S1.2
Changed lines of the file:
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@@
 <part name="J1" library="SparkFun-Connectors" deviceset="CONN_14" device="LONGPADS"/>
 <part name="R1" library="resistor" library_urn="urn:adsk.eagle:library:348" deviceset="R-EU_" device="0204/5" package3d_urn="urn:adsk.eagle:package:25955/1"/>
+<part name="S1" library="SparkFun-Switches" deviceset="MOMENTARY-SWITCH-SPST" device="-PTH-6.0MM-KIT"/>
 </parts>
 <sheets>
@@
 <instance part="J1" gate="G$1" x="147.32" y="114.3" rot="R270"/>
 <instance part="R1" gate="G$1" x="30.48" y="91.44" rot="R90"/>
+<instance part="S1" gate="G$1" x="116.84" y="-30.48"/>
 </instances>
 <busses>
@@
 <pinref part="JP4" gate="G$1" pin="1"/>
 <wire x1="111.76" y1="43.18" x2="127" y2="43.18" width="0.1524" layer="91"/>
+<pinref part="S1" gate="G$1" pin="2"/>
+<wire x1="121.92" y1="-30.48" x2="121.92" y2="2.54" width="0.1524" layer="91"/>
+<wire x1="121.92" y1="2.54" x2="111.76" y2="2.54" width="0.1524" layer="91"/>
+<junction x="111.76" y="2.54"/>
 </segment>
 </net>
@@
 </segment>
 </net>
+<net name="N$18" class="0">
+<segment>
+<pinref part="S1" gate="G$1" pin="1"/>
+<wire x1="111.76" y1="-30.48" x2="68.58" y2="-30.48" width="0.1524" layer="91"/>
+<wire x1="68.58" y1="-30.48" x2="68.58" y2="55.88" width="0.1524" layer="91"/>
+<pinref part="ARDUINO1" gate="G$1" pin="RST"/>
+<wire x1="68.58" y1="55.88" x2="53.34" y2="55.88" width="0.1524" layer="91"/>
+</segment>
+</net>

Commit message: Add files via upload
Parts:
- removed J1: (no value), SparkFun-Connectors:CONN_14LONGPADS
- removed S1: MOMENTARY-SWITCH-SPST-PTH-6.0MM-KIT, SparkFun-Switches:MOMENTARY-SWITCH-SPST-PTH-6.0MM-KIT
- removed X3: 22-23-2041, con-molex:22-23-2041
- added JP7: (no value), adafruit:PINHD-1X1
- added JP8: (no value), adafruit:PINHD-1X14-CB
- added JP9: (no value), adafruit:PINHD-1X3
Connections:
- removed net N$18: ARDUINO1.RST, S1.1
- removed net N$3 (its old number): ARDUINO1.VCC, J1.1, J1.4, J1.8, JP3.1, R1.1, U$1.RST, U$1.VCC, X3-1.S
- removed net N$4: ARDUINO1.GND, J1.2, JP4.1, S1.2, U$1.GND, X3-4.S
- new net GND: ARDUINO1.GND, JP4.1, JP8.2, JP9.3, U$1.GND
- new net VCC: ARDUINO1.VCC, JP3.1, JP8.1, JP8.4, JP8.8, JP9.1, R1.1, U$1.CH_PD, U$1.VCC
- net N$11: now also JP8.6; no longer J1.6
- net N$12: now also JP8.9; no longer J1.9
- net N$13: now also JP8.10; no longer J1.10
- net N$14: now also JP8.11; no longer J1.11
- net N$15: now also JP8.12; no longer J1.12
- net N$16: now also JP8.13; no longer J1.13
- net N$17: now also JP8.14; no longer J1.14
- net N$5: now also JP8.3; no longer J1.3
- net N$6: now also JP9.2; no longer X3-2.S
- net N$7: now also JP8.7; no longer J1.7
- net N$8: now also JP8.5; no longer J1.5
